Commit message: bug_fix

File: my_mobile/urdf/macros.xacro (robot description, xacro)
@@ -1,5 +1,5 @@
 <?xml version="1.0"?>
-<robot>
-    <macro name="link_wheel" params="name">
+<robot xmlns:xacro="http://www.ros.org/wiki/xacro">
+    <xacro:macro name="link_wheel" params="name">
         <link name="${name}">
             <inertial>
@@ -21,6 +21,6 @@
             </visual>
         </link>
-    </macro>
-    <macro name="joint_wheel" params="name child origin_xyz">
+    </xacro:macro>
+    <xacro:macro name="joint_wheel" params="name child origin_xyz">
       <joint name="${name}" type="continuous">
         <origin rpy="0 0 0" xyz="${origin_xyz}"/>
@@ -31,4 +31,4 @@
         <joint_properties damping="1.0" friction="1.0"/>
       </joint>
-    </macro>
+    </xacro:macro>
 </robot>
